File: kicad/WristMountedPhaser/WristMountedPhaser.kicad_pcb (KiCad board)
At the start: 2 copper layers, 28.3 x 38.1 mm, 37 parts

Commit message: added instructions to kicad text
Other:
- board text added: "5v (150R) 3v (100R) Solder in order:"
- board text added: "Acceptable voltage: 3v3 to 5v"
- board text added: "VCC"
- board text removed: "+5v"
- board text removed: "All Resistors are 150R Solder in order:"
Changed lines of the file:
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@@
 		)
 	)
-	(gr_text "+5v"
+	(gr_text "VCC"
 		(at 48.468547 34.15 90)
 		(layer "F.SilkS")
@@
 		)
 	)
-	(gr_text "+5v"
+	(gr_text "VCC"
 		(at 48.468547 40.59 90)
 		(layer "F.SilkS")
@@
 		)
 	)
-	(gr_text "+5v"
+	(gr_text "Acceptable voltage: 3v3 to 5v"
+		(at 43.37 49.77 0)
+		(layer "B.SilkS")
+		(effects
+			(font
+				(size 0.8 0.8)
+				(thickness 0.15)
+			)
+			(justify left bottom mirror)
+		)
+	)
+	(gr_text "An ATTiny 402 may be used \ninstead of a Wemos D1 mini"
+		(at 43.37 52.4 0)
+		(layer "B.SilkS")
+		(effects
+			(font
+				(size 0.8 0.8)
+				(thickness 0.15)
+			)
+			(justify left bottom mirror)
+		)
+	)
+	(gr_text "VCC"
 		(at 39.92 28.2 0)
 		(layer "B.SilkS")
@@
 		)
 	)
-	(gr_text "All Resistors are 150R\n\nSolder in order:"
-		(at 38.62 32.39 0)
+	(gr_text "5v (150R) 3v (100R)\nSolder in order:"
+		(at 39.6 32.16 0)
 		(layer "B.SilkS")
 		(effects
-			(font
-				(size 1 1)
-				(thickness 0.15)
-			)
-			(justify left bottom mirror)
-		)
-	)
-	(gr_text "An ATTiny 402 may be used \ninstead of a Wemos D1 mini"
-		(at 42.96 51.57 0)
-		(layer "B.SilkS")
-		(effects

Commit message: added instructions to kicad text
Other:
- board text added: "5v (150R) 3v3 (100R) Solder in order:"
- board text removed: "5v (150R) 3v (100R) Solder in order:"
Changed lines of the file:
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@@
+		)
+	)
+	(gr_text "5v (150R) 3v3 (100R)\nSolder in order:"
+		(at 38.62 32.16 0)
+		(layer "B.SilkS")
+		(effects
+			(font
+				(size 0.8 0.8)
+				(thickness 0.15)
+			)
+			(justify left bottom mirror)
 		)
 	)
@@
 		(layer "B.SilkS")
 		(effects
-			(font
-				(size 1 1)
-				(thickness 0.15)
-			)
-			(justify left bottom mirror)
-		)
-	)
-	(gr_text "5v (150R) 3v (100R)\nSolder in order:"
-		(at 39.6 32.16 0)
-		(layer "B.SilkS")
-		(effects
